File: Hardware/SparkFun GPS NEO_M9N_SMA/SparkFun GPS NEO_M9N_SMA.brd (EAGLE design)
At the start: 40.6 x 36.8 mm, 94 parts, among them J2 Qwiic Right Angle, J4 Qwiic Right Angle, U1 U-BLOX_NEO-M9N, U2 3.3V

Commit message: Changes to female SMD, SMA connector
Parts:
- E1: value ANTENNA-GROUNDEDEDGE_RPSMA_SMD -> ANTENNA-GROUNDEDEDGE_SMA_SMD
Changed lines of the file:
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@@
 <layer number="25" name="tNames" color="7" fill="1" visible="no" active="yes"/>
 <layer number="26" name="bNames" color="7" fill="1" visible="no" active="yes"/>
-<layer number="27" name="tValues" color="7" fill="1" visible="no" active="yes"/>
+<layer number="27" name="tValues" color="7" fill="1" visible="yes" active="yes"/>
 <layer number="28" name="bValues" color="7" fill="1" visible="no" active="yes"/>
 <layer number="29" name="tStop" color="7" fill="3" visible="no" active="yes"/>
@@
 <element name="U$14" library="SparkFun-Aesthetics" package="QWIIC_4MM" value="" x="2.286" y="11.176" smashed="yes"/>
 <element name="U$21" library="NEO_GPS_board_silk_FINAL#03#jpg" package="NEO_GPS_BOARD_SILK_FINAL#03#JPG" value="" x="15.24" y="11.43" smashed="yes" rot="MR0"/>
-<element name="E1" library="SparkFun-RF" package="SMA-EDGE-SMD" value="ANTENNA-GROUNDEDEDGE_RPSMA_SMD" x="40.4114" y="25.654" smashed="yes" rot="R270">
-<attribute name="PROD_ID" value="CONN-15101" x="40.4114" y="25.654" size="1.778" layer="27" font="vector" ratio="15" rot="R270" display="off"/>
+<element name="E1" library="SparkFun-RF" package="SMA-EDGE-SMD" value="ANTENNA-GROUNDEDEDGE_SMA_SMD" x="40.4114" y="25.654" smashed="yes" rot="R270">
+<attribute name="PROD_ID" value="CONN-15100" x="40.4114" y="25.654" size="1.778" layer="27" font="vector" ratio="15" rot="R270" display="off"/>
 </element>
 <element name="FB1" library="SparkFun-Coils" package="0402" value="FERRITE_BEAD-120_OHM-0402" x="28.3972" y="21.5138" smashed="yes" rot="R270">
